File: 40pin_1.27mm_to_20pin_2.54mm.kicad_pcb (KiCad board)
At the start: 2 copper layers, 2 parts, among them J1 Conn_02x20_Odd_Even, J2 Conn_02x10_Odd_Even

Commit message: Add files via upload
Other:
- board outline added: 10.2 x 26.7 mm
Changed lines of the file:
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@@
       (drillshape 0)
       (scaleselection 1)
-      (outputdirectory "out/pos")
+      (outputdirectory "out/gerbers")
     )
   )
@@
     )
   )
+  (gr_rect (start -5.08 13.335) (end 5.08 -13.335) (layer "Edge.Cuts") (width 0.1) (fill none))
   (segment (start -4.110103 0.724511) (end -4.534511 0.300103) (width 0.25) (layer "F.Cu") (net 1))
   (segment (start -2.840103 0.724511) (end -4.110103 0.724511) (width 0.25) (layer "F.Cu") (net 1))
